Commit message: Use a box for feet collision

File: urdf/darwin.urdf (robot description, URDF)
Before this commit: robot darwinOP, 27 links, 26 joints
Links:
- link MP_ANKLE2_L: geometry collision box size=0.004 0.035 0.090; visual mesh filename=package://darwin_description/meshes/ankle2_l.STL scale=1 1 1
- link MP_ANKLE2_R: geometry collision box size=0.004 0.035 0.090; visual mesh filename=package://darwin_description/meshes/ankle2_r.STL scale=1 1 1
